File: reviung34/pcb/reviung34-orig.kicad_pcb (KiCad board)
At the start: 2 copper layers, 214.3 x 107.1 mm, 95 parts, among them SW1 SW_PUSH, SW10 SW_PUSH, SW11 SW_PUSH, SW12 SW_PUSH, SW13 SW_PUSH, SW14 SW_PUSH, SW15 SW_PUSH, SW16 SW_PUSH, SW17 SW_PUSH, SW18 SW_PUSH, SW19 SW_PUSH, SW2 SW_PUSH, SW20 SW_PUSH, SW21 SW_PUSH, SW22 SW_PUSH, SW23 SW_PUSH, SW24 SW_PUSH, SW25 SW_PUSH, SW26 SW_PUSH, SW27 SW_PUSH, SW28 SW_PUSH, SW29 SW_PUSH, SW3 SW_PUSH, SW30 SW_PUSH, SW31 SW_PUSH, SW32 SW_PUSH, SW33 SW_PUSH, SW34 SW_PUSH, SW35 SW_PUSH, SW4 SW_PUSH, SW5 SW_PUSH, SW6 SW_PUSH, SW7 SW_PUSH, SW8 SW_PUSH, SW9 SW_PUSH, U1 ProMicro

Commit message: using kbd switches and pro-micro
Connections:
- U1 pad 1: GND -> LED
- U1 pad 10: Net-(U1-Pad10) -> col3
- U1 pad 11: Net-(U1-Pad11) -> col4
- U1 pad 13: Net-(U1-Pad13) -> col8
- U1 pad 14: Net-(U1-Pad14) -> col7
- U1 pad 15: col8 -> col6
- U1 pad 16: col7 -> col5
- U1 pad 17: col6 -> row3
- U1 pad 18: col5 -> row2
- U1 pad 19: row3 -> row1
- U1 pad 2: GND -> Net-(U1-Pad2)
- U1 pad 20: row2 -> row0
- U1 pad 21: row1 -> VCC
- U1 pad 22: row0 -> reset
- U1 pad 23: VCC -> GND
- U1 pad 24: reset -> Net-(U1-Pad24)
- U1 pad 3: Net-(U1-Pad3) -> GND
- U1 pad 4: Net-(U1-Pad4) -> GND
- U1 pad 5: col0 -> Net-(U1-Pad5)
- U1 pad 6: col1 -> Net-(U1-Pad6)
- U1 pad 7: col2 -> col0
- U1 pad 8: col3 -> col1
- U1 pad 9: col4 -> col2
