File: reviung34/pcb/reviung34.sch (KiCad schematic (older format))
At the start: 80 parts, among them SW1 SW_PUSH, SW10 SW_PUSH, SW11 SW_PUSH, SW12 SW_PUSH, SW13 SW_PUSH, SW14 SW_PUSH, SW15 SW_PUSH, SW16 SW_PUSH, SW17 SW_PUSH, SW18 SW_PUSH, SW19 SW_PUSH, SW2 SW_PUSH, SW20 SW_PUSH, SW21 SW_PUSH, SW22 SW_PUSH, SW23 SW_PUSH, SW24 SW_PUSH, SW25 SW_PUSH, SW26 SW_PUSH, SW27 SW_PUSH, SW28 SW_PUSH, SW29 SW_PUSH, SW3 SW_PUSH, SW30 SW_PUSH, SW31 SW_PUSH, SW32 SW_PUSH, SW33 SW_PUSH, SW34 SW_PUSH, SW35 SW_PUSH, SW4 SW_PUSH, SW5 SW_PUSH, SW6 SW_PUSH, SW7 SW_PUSH, SW8 SW_PUSH, SW9 SW_PUSH, U1 ProMicro

Commit message: using kbd switches and pro-micro
Parts:
- RESET1, SW8: symbol _reviung-kbd:SW_PUSH -> reviung34-rescue:SW_PUSH-_reviung-kbd
- SW1, SW10, SW11, SW12, SW13, SW14, SW15, SW16, SW17, SW18, SW19, SW2, SW20, SW21, SW22, SW23, SW24, SW25, SW26, SW27, SW28, SW29, SW3, SW30, SW31, SW32, SW33, SW34, SW35, SW4, SW5, SW6, SW7, SW9: symbol _reviung-kbd:SW_PUSH -> kbd:SW_PUSH
- U1: symbol _reviung-kbd:ProMicro -> kbd:ProMicro
Changed lines of the file:
@@
 $EndComp
 $Comp
-L _reviung-kbd:ProMicro U1
+L kbd:ProMicro U1
 U 1 1 6051A543
 P 1800 5950
@@
 NoConn ~ 2500 5200
 $Comp
-L _reviung-kbd:SW_PUSH RESET1
+L reviung34-rescue:SW_PUSH-_reviung-kbd RESET1
 U 1 1 6051CE8E
 P 5000 7300
@@
 NoConn ~ 9100 5500
 $Comp
-L _reviung-kbd:SW_PUSH SW1
+L kbd:SW_PUSH SW1
 U 1 1 6052930F
 P 1500 1500
@@
 $EndComp
 $Comp
-L _reviung-kbd:SW_PUSH SW6
+L kbd:SW_PUSH SW6
 U 1 1 6052B601
 P 1500 2150
@@
 $EndComp
 $Comp
-L _reviung-kbd:SW_PUSH SW11
+L kbd:SW_PUSH SW11
 U 1 1 6052CF4B
 P 1500 2800
@@
 $EndComp
 $Comp
-L _reviung-kbd:SW_PUSH SW2
+L kbd:SW_PUSH SW2
 U 1 1 60530877
 P 2600 1500
@@
 $EndComp
 $Comp
-L _reviung-kbd:SW_PUSH SW7
+L kbd:SW_PUSH SW7
 U 1 1 60530883
 P 2600 2150
@@
 $EndComp
 $Comp
-L _reviung-kbd:SW_PUSH SW12
+L kbd:SW_PUSH SW12
 U 1 1 6053088F
 P 2600 2800
@@
 $EndComp
 $Comp
-L _reviung-kbd:SW_PUSH SW3
+L kbd:SW_PUSH SW3
 U 1 1 60536207
 P 3700 1500
@@
 $EndComp
 $Comp
-L _reviung-kbd:SW_PUSH SW8
+L reviung34-rescue:SW_PUSH-_reviung-kbd SW8
 U 1 1 60536213
 P 3700 2150
@@
 $EndComp
 $Comp
-L _reviung-kbd:SW_PUSH SW13
+L kbd:SW_PUSH SW13
 U 1 1 6053621F
 P 3700 2800
@@
 $EndComp
 $Comp
-L _reviung-kbd:SW_PUSH SW4
+L kbd:SW_PUSH SW4
 U 1 1 6053622B
 P 4800 1500
@@
 $EndComp
 $Comp
-L _reviung-kbd:SW_PUSH SW9
+L kbd:SW_PUSH SW9
 U 1 1 60536237
 P 4800 2150
@@
 $EndComp
 $Comp
-L _reviung-kbd:SW_PUSH SW14
+L kbd:SW_PUSH SW14
 U 1 1 60536243
 P 4800 2800
@@
 $EndComp
 $Comp
-L _reviung-kbd:SW_PUSH SW5
+L kbd:SW_PUSH SW5
 U 1 1 60540B4F
 P 5900 1500
@@
 $EndComp
 $Comp
-L _reviung-kbd:SW_PUSH SW10
+L kbd:SW_PUSH SW10
 U 1 1 60540B5B
 P 5900 2150
@@
 $EndComp
 $Comp
-L _reviung-kbd:SW_PUSH SW15
+L kbd:SW_PUSH SW15
 U 1 1 60540B67
 P 5900 2800
@@
 $EndComp
 $Comp
-L _reviung-kbd:SW_PUSH SW19
+L kbd:SW_PUSH SW19
 U 1 1 60540B73
 P 7000 1500
@@
 $EndComp
 $Comp
-L _reviung-kbd:SW_PUSH SW23
+L kbd:SW_PUSH SW23
 U 1 1 60540B7F
 P 7000 2150
@@
 $EndComp
 $Comp
-L _reviung-kbd:SW_PUSH SW27
+L kbd:SW_PUSH SW27
 U 1 1 60540B8B
 P 7000 2800
@@
 $EndComp
 $Comp
-L _reviung-kbd:SW_PUSH SW20
+L kbd:SW_PUSH SW20
 U 1 1 60540B97
 P 8100 1500
@@
 $EndComp
 $Comp
-L _reviung-kbd:SW_PUSH SW24
+L kbd:SW_PUSH SW24
 U 1 1 60540BA3
 P 8100 2150
@@
 $EndComp
 $Comp
-L _reviung-kbd:SW_PUSH SW28
+L kbd:SW_PUSH SW28
 U 1 1 60540BAF
 P 8100 2800
@@
 $EndComp
 $Comp
-L _reviung-kbd:SW_PUSH SW21
+L kbd:SW_PUSH SW21
 U 1 1 60540BBB
 P 9200 1500
@@
 $EndComp
 $Comp
-L _reviung-kbd:SW_PUSH SW25
+L kbd:SW_PUSH SW25
 U 1 1 60540BC7
 P 9200 2150
@@
 $EndComp
 $Comp
-L _reviung-kbd:SW_PUSH SW29
+L kbd:SW_PUSH SW29
 U 1 1 60540BD3
 P 9200 2800
@@
 $EndComp
 $Comp
-L _reviung-kbd:SW_PUSH SW22
+L kbd:SW_PUSH SW22
 U 1 1 60544E37
 P 10300 1500
@@
 $EndComp
 $Comp
-L _reviung-kbd:SW_PUSH SW26
+L kbd:SW_PUSH SW26
 U 1 1 60544E43
 P 10300 2150
@@
 $EndComp
 $Comp
-L _reviung-kbd:SW_PUSH SW30
+L kbd:SW_PUSH SW30
 U 1 1 60544E4F
 P 10300 2800
@@
 $EndComp
 $Comp
-L _reviung-kbd:SW_PUSH SW35
+L kbd:SW_PUSH SW35
 U 1 1 6054F871
 P 6450 3800
@@
 $EndComp
 $Comp
-L _reviung-kbd:SW_PUSH SW16
+L kbd:SW_PUSH SW16
 U 1 1 6054F87D
 P 3700 3450
@@
 $EndComp
 $Comp
-L _reviung-kbd:SW_PUSH SW17
+L kbd:SW_PUSH SW17
 U 1 1 6054F889
 P 4800 3450
@@
 $EndComp
 $Comp
-L _reviung-kbd:SW_PUSH SW18
+L kbd:SW_PUSH SW18
 U 1 1 6054F895
 P 5750 3800
@@
 $EndComp
 $Comp
-L _reviung-kbd:SW_PUSH SW31
+L kbd:SW_PUSH SW31
 U 1 1 6054F8A1
 P 7000 3450
@@
 $EndComp
 $Comp
-L _reviung-kbd:SW_PUSH SW32
+L kbd:SW_PUSH SW32
 U 1 1 6054F8AD
 P 8100 3450
@@
 $EndComp
 $Comp
-L _reviung-kbd:SW_PUSH SW33
+L kbd:SW_PUSH SW33
 U 1 1 6054F8B9
 P 9200 3450
@@
 $EndComp
 $Comp
-L _reviung-kbd:SW_PUSH SW34
+L kbd:SW_PUSH SW34
 U 1 1 6054F8C5
 P 10300 3450

Commit message: choc version of r34
Parts:
- removed D12, D14, D17, D19, D2, D22, D23, D26, D27, D30, D32, D34, D4, D7, D9: 1N4148W, _reviung-kbd:D3_SMD_1side, symbol Diode:1N4148W
- D1, D10, D11, D13, D15, D16, D18, D20, D21, D24, D25, D28, D29, D3, D31, D33, D5, D6, D8: value 1N4148W -> BAV70; footprint _reviung-kbd:D3_SMD_1side -> Package_TO_SOT_SMD:SOT-23; symbol Diode:1N4148W -> Diode:BAV70
- RESET1: footprint _reviung-kbd:ResetSW_1side -> kbd-footprints:ResetSW_1side
- RGB1, RGB2, RGB3, RGB4, RGB5, RGB6, RGB7, RGB8, RGB9: footprint _reviung-kbd:LED_WS2812B_PLCC4_5.0x5.0mm_P3.2mm -> LED_SMD:LED_WS2812B_PLCC4_5.0x5.0mm_P3.2mm
- SW1, SW10, SW11, SW12, SW13, SW14, SW15, SW16, SW19, SW2, SW20, SW21, SW22, SW23, SW24, SW25, SW26, SW27, SW28, SW29, SW3, SW30, SW31, SW32, SW33, SW34, SW4, SW5, SW6, SW7, SW8, SW9: footprint _reviung-kbd:MXOnly-1U-NoLED -> kbd-footprints:CherryMX_Choc_1u
- SW17: footprint _reviung-kbd:MXOnly-1U-5pinRcut -> kbd-footprints:CherryMX_Choc_1u
- SW18: footprint _reviung-kbd:MXOnly-1U-5pinLcut -> kbd-footprints:CherryMX_Choc_1u
- SW35: footprint _reviung-kbd:MXOnly-2U-NoLED-or1Ux2 -> Keebio-Parts:Kailh-PG1350-1u-NoLED
- U1: footprint _reviung-kbd:ProMicro -> kbd-footprints:ProMicro_v3
Connections:
- net GND: now also U1.23 (GND), U1.3 (GND), U1.4 (GND); no longer U1.1 (TX0/D3), U1.2 (RX1/D2)
- net LED: now also U1.1 (TX0/D3)
- net VCC: now also U1.21 (VCC); no longer U1.23 (GND)
- net col0: now also SW1.2, SW11.2, SW6.2, U1.7 (4/D4); no longer SW1.1, SW11.1, SW6.1, U1.5 (2/D1/SDA)
- net col1: now also U1.8 (5/C6); no longer U1.6 (3/D0/SCL)
- net col2: now also SW13.2, SW3.2, SW8.2, U1.9 (6/D7); no longer SW13.1, SW3.1, SW8.1, U1.7 (4/D4)
- net col3: now also SW17.2, U1.10 (7/E6); no longer SW17.1, U1.8 (5/C6)
- net col4: now also SW10.2, SW15.2, SW5.2, U1.11 (8/B4); no longer SW10.1, SW15.1, SW5.1, U1.9 (6/D7)
- net col5: now also U1.16 (B1/15); no longer U1.18 (F6/A1)
- net col6: now also SW20.2, SW24.2, SW28.2, U1.15 (B3/14); no longer SW20.1, SW24.1, SW28.1, U1.17 (F7/A0)
- net col7: now also U1.14 (B2/16); no longer U1.16 (B1/15)
- net col8: now also SW22.2, SW26.2, SW30.2, SW34.2, U1.13 (B6/10); no longer SW22.1, SW26.1, SW30.1, SW34.1, U1.15 (B3/14)
- net reset: now also U1.22 (RST); no longer U1.24 (RAW)
- net row0: now also D1.3 (K), D20.3 (K), D21.3 (K), D3.3 (K), D5.3 (K), U1.20 (F4/A3); no longer D1.1 (K), D20.1 (K), D21.1 (K), D3.1 (K), D5.1 (K), U1.22 (RST)
- net row1: now also D10.3 (K), D24.3 (K), D25.3 (K), D6.3 (K), D8.3 (K), U1.19 (F5/A2); no longer D10.1 (K), D24.1 (K), D25.1 (K), D6.1 (K), D8.1 (K), U1.21 (VCC)
- net row2: now also D11.3 (K), D13.3 (K), D15.3 (K), D28.3 (K), D29.3 (K), U1.18 (F6/A1); no longer D11.1 (K), D13.1 (K), D15.1 (K), D28.1 (K), D29.1 (K), U1.20 (F4/A3)
- net row3: now also D16.3 (K), D18.3 (K), D31.3 (K), D33.3 (K), U1.17 (F7/A0); no longer D16.1 (K), D18.1 (K), D31.1 (K), D33.1 (K), U1.19 (F5/A2)
- net at D1.2 (A): now also D1.1 (A), SW1.1; no longer SW1.2
- net at D6.2 (A): now also D6.1 (A), SW6.1; no longer SW6.2
- net at D11.2 (A): now also D11.1 (A), SW11.1; no longer SW11.2
- net at SW2.2: now also D3.1 (A)
- net at SW7.2: now also D8.1 (A)
- net at SW12.2: now also D13.2 (A)
- net at D3.2 (A): now also SW3.1; no longer SW3.2
- net at D8.2 (A): now also SW8.1; no longer SW8.2
- net at SW4.2: now also D5.1 (A)
- net at SW9.2: now also D10.2 (A)
- net at SW14.2: now also D15.2 (A)
- net at D5.2 (A): now also SW5.1; no longer SW5.2
- net at SW19.2: now also D20.1 (A)
- net at SW23.2: now also D24.1 (A)
- net at SW27.2: now also D28.2 (A)
- net at D20.2 (A): now also SW20.1; no longer SW20.2
- net at D24.2 (A): now also SW24.1; no longer SW24.2
- net at SW21.2: now also D21.1 (A); no longer D21.2 (A)
- net at SW25.2: now also D25.1 (A); no longer D25.2 (A)
- net at SW18.2, SW35.2: now also D18.1 (A); no longer D18.2 (A)
- net at SW16.2: now also D16.1 (A); no longer D16.2 (A)
- net at SW32.2: now also D31.1 (A)
- net at D33.2 (A), SW33.2: now also D33.1 (A)
- new net: D13.1 (A), SW13.1
- new net: D10.1 (A), SW10.1
- new net: D15.1 (A), SW15.1
- new net: D28.1 (A), SW28.1
- new net: D21.2 (A), SW22.1
- new net: D25.2 (A), SW26.1
- new net: D29.1 (A), SW30.1
- new net: D16.2 (A), SW17.1
- new net: D18.2 (A), SW34.1
Other:
- moved on the sheet: SW1, SW10, SW11, SW12, SW13, SW14, SW15, SW16, SW17, SW18, SW19, SW2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
